File: comm_module.kicad_sch (KiCad schematic)
At the start: 80 parts, among them J1 USB-231-ARY, J2 PH2.54-01-03PZS, J3 U.FL-R-SMT-1(80), J4 U.FL-R-SMT-1(80), J5 U.FL-R-SMT-1(80), J6 U.FL-R-SMT-1(80), J7 S3B-ZR-SM4A-TF(LF)(SN), J8 SMN-305-ARP7, J9 U.FL-R-SMT-1(80), Q1 BSS138PW,115, U1 MIC29302WU, U2 SIM7600E, U3 TXU0202DCUR, U4 TCA9406DCUR, X1 WJ500V-5.08-2P-14-00A

Commit message: First no error draft
Parts:
- removed C12, C14: GRM0335C1H100JA01D, pepy_sym_lib:[CAP_SMD_0201_0603Metric], symbol pepy_sym_lib:[CAP_SMD_0201_0603Metric]muRata GRM0335C1H100JA01D
- removed C16: CC1206KKX7RDBB102, pepy_sym_lib:[CAP_SMD_1206_3216Metric], symbol pepy_sym_lib:[CAP_SMD_1206_3216Metric]YAGEO CC1206KKX7RDBB102
- removed J2: PH2.54-01-03PZS, pepy_sym_lib:[2x3_PIN_HEADER_STR]XUNPU PH2.54-01-03PZS, symbol pepy_sym_lib:[2x3_PIN_HEADER_STR]XUNPU PH2.54-01-03PZS
- removed J7: S3B-ZR-SM4A-TF(LF)(SN), pepy_sym_lib:[JST_1X3P_1_5MM_R_ANGLE]JST S3B-ZR-SM4A-TF(LF)(SN), symbol pepy_sym_lib:[JST_1X3P_1_5MM_R_ANGLE]JST S3B-ZR-SM4A-TF(LF)(SN)
- removed R10: RC0201FR-0733RL, pepy_sym_lib:[RES_SMD_0201_0603Metric], symbol pepy_sym_lib:[RES_SMD_0201_0603Metric]YAGEO RC0201FR-0733RL
- removed R12, R2, R8: 0402WGF0000TCE, pepy_sym_lib:[RES_SMD_0402_1005Metric], symbol pepy_sym_lib:[RES_SMD_0402_1005Metric]UNI-ROYAL(Uniroyal Elec) 0402WGF0000TCE
- removed R15: 0805W8F1004T5E, pepy_sym_lib:[RES_SMD_0805_2012Metric], symbol pepy_sym_lib:[RES_SMD_0805_2012Metric]UNI-ROYAL(Uniroyal Elec) 0805W8F1004T5E
- removed R20: 0201WMF1002TEE, pepy_sym_lib:[RES_SMD_0201_0603Metric], symbol pepy_sym_lib:[RES_SMD_0201_0603Metric]UNI-ROYAL(Uniroyal Elec) 0201WMF1002TEE
- removed R6: RC0201FR-071ML, pepy_sym_lib:[RES_SMD_0201_0603Metric], symbol pepy_sym_lib:[RES_SMD_0201_0603Metric]YAGEO RC0201FR-071ML
- added C13, C15: GRM0335C1H100JA01D, pepy_sym_lib:[CAP_SMD_0201_0603Metric], symbol pepy_sym_lib:[CAP_SMD_0201_0603Metric]muRata GRM0335C1H100JA01D
- added C16, C6: CC0201KRX5R6BB104, pepy_sym_lib:[CAP_SMD_0201_0603Metric], symbol pepy_sym_lib:[CAP_SMD_0201_0603Metric]YAGEO CC0201KRX5R6BB104
- added C22: CC0402KRX7R7BB104, pepy_sym_lib:[CAP_SMD_0402_1005Metric], symbol pepy_sym_lib:[CAP_SMD_0402_1005Metric]YAGEO CC0402KRX7R7BB104
- added J2: PZ254V-11-06P, pepy_sym_lib:[6P_HEADER_STR]XFCN PZ254V-11-06P, symbol pepy_sym_lib:[6P_HEADER_STR]XFCN PZ254V-11-06P
- added R10, R7: 0402WGF0000TCE, pepy_sym_lib:[RES_SMD_0402_1005Metric], symbol pepy_sym_lib:[RES_SMD_0402_1005Metric]UNI-ROYAL(Uniroyal Elec) 0402WGF0000TCE
- added R15, R17, R19, R20: 0805W8F0000T5E, pepy_sym_lib:[RES_SMD_0805_2012Metric], symbol pepy_sym_lib:[RES_SMD_0805_2012Metric]UNI-ROYAL(Uniroyal Elec) 0805W8F0000T5E
- added R21, R22, R23, R24: 0402WGF2201TCE, pepy_sym_lib:[RES_SMD_0402_1005Metric], symbol pepy_sym_lib:[RES_SMD_0402_1005Metric]UNI-ROYAL(Uniroyal Elec) 0402WGF2201TCE
- added R5: 0805W8F1004T5E, pepy_sym_lib:[RES_SMD_0805_2012Metric], symbol pepy_sym_lib:[RES_SMD_0805_2012Metric]UNI-ROYAL(Uniroyal Elec) 0805W8F1004T5E
- added TP6: nRST, pepy_sym_lib:[TEST_POINT]TestPoint_Pad_D1.0mm, symbol Connector:TestPoint
- J3, J4, J5, J6: value U.FL-R-SMT-1(80) -> U.FLRSMT1
- J8: renamed from J9; value U.FL-R-SMT-1(80) -> U.FLRSMT1
- TP1, TP2, TP3, TP4, TP5: footprint (none) -> pepy_sym_lib:[TEST_POINT]TestPoint_Pad_D1.0mm
- TP7: renamed from TP6; footprint (none) -> pepy_sym_lib:[TEST_POINT]TestPoint_Pad_D1.0mm
- renumbered C9 to C10, C10 to C11, C11 to C12, C13 to C14, C15 to C17, C17 to C18, C18 to C19, C19 to C20, C20 to C21, C21 to C23, C22 to C24, C23 to C25, C24 to C26, C25 to C27, C6 to C7, C7 to C8, C8 to C9, J8 to J7, R13 to R11, R14 to R12, R16 to R13, R17 to R14, R18 to R16, R19 to R18, R3 to R2, R21 to R25, R22 to R26, R23 to R27, R4 to R3, R5 to R4, R7 to R6, R9 to R8, R11 to R9
Connections:
- net NETFLIGHT is gone; now on net NETLIGHT: Q1.1 (G), R25.2, R26.2
- net 1V8_COMM: now also C11.2, U3.3 (VCCA), U3.6 (OE), U4.6 (OE), C6.2, R15.2, R21.2, R22.2; no longer C17.2, R13.2, U3.7 (VCCB)
- net AUX_ANT: now also C13.2, R7.1
- net COMM_SCL: now also R22.1
- net COMM_SDA: now also R21.1
- net Earth_USB: now also R5.1
- net GND: now also C13.1, C15.1, C16.1, C22.1, C6.1, J2.1, R5.2
- net MAIN_ANT: now also C12.2, R6.1
- net M_RX_S_TX: now also U3.8 (B1Y), J2.5; no longer U3.4 (A2Y)
- net M_RX_S_TX_1V8: now also U3.5 (A1); no longer U3.1 (B2)
- net M_TX_S_RX: now also U3.1 (B2), J2.6; no longer U3.5 (A1)
- net M_TX_S_RX_1V8: now also U3.4 (A2Y); no longer U3.8 (B1Y)
- net SCL: now also J2.3, R24.1
- net SDA: now also J2.2, R23.1
- net SIM_CLK: now also D5.4; no longer D5.5
- net SIM_DATA: now also D5.5; no longer D5.1
- net SIM_RST: now also D5.3; no longer D5.4
- net SIM_VCC: now also D5.1, U2.20 (USIM_VDD), C16.2; no longer D5.3, R16.2
- net VBUS: now also R19.2
- net VDD_3V3: now also C17.2, U3.7 (VCCB), J2.4, R17.2, R23.2, R24.2; no longer C11.2, R27.2, U3.3 (VCCA), U3.6 (OE)
- net VDD_COMM: now also R27.2, R20.2
- net DFILT-: now reaches D3.1 (I/O1), L1.2
- net DFILT+: now reaches D3.3 (I/O2), L1.3
- net at J8.1: now also C20.2, L4.1
- net at J5.1: now also R9.2
- net at J6.1: now also R10.2
- net VDD_AUX: now reaches U2.44 (VDD_AUX)
- net VDD_AUX: now also R13.2
- net D+_COMM renamed DCOMM+
- net D-_COMM renamed DCOMM-
- net nRST: no longer names the net of U2.4 (RESET)
- net nRST: now also TP6.1
- new net: C22.2, R15.1, R16.2, R17.1, R19.1, R20.1
- new net: C15.2, R10.1, R7.2
- no-connect marks 38 -> 37
Other:
- note added: "VDD_3V3 hier ENable"
- moved on the sheet: C12, C26, C27, R6, U4
