File: comm_module.kicad_sch (KiCad schematic)
At the start: 86 parts, among them J1 USB-231-ARY, J2 PZ254V-11-06P, J3 U.FLRSMT1, J4 U.FLRSMT1, J5 U.FLRSMT1, J6 U.FLRSMT1, J7 SMN-305-ARP7, J8 U.FLRSMT1, Q1 BSS138PW,115, U1 MIC29302WU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

Commit message: Antenna polygon fixes and refinements
Parts:
- added C28: CC0201KRX5R6BB104, pepy_sym_lib:[CAP_SMD_0201_0603Metric], symbol pepy_sym_lib:[CAP_SMD_0201_0603Metric]YAGEO CC0201KRX5R6BB104
- added D7, D8, D9: ESD56151W05, pepy_sym_lib:[ESD_PROT]WILLSEMI ESD56151W05-2TR, symbol pepy_sym_lib:[ESD_PROT]WILLSEMI ESD56151W05-2TR
- added R28, R29: 0402WGF0000TCE, pepy_sym_lib:[RES_SMD_0402_1005Metric], symbol pepy_sym_lib:[RES_SMD_0402_1005Metric]UNI-ROYAL(Uniroyal Elec) 0402WGF0000TCE
- added TP10: 1V8_COMM, pepy_sym_lib:[TEST_POINT]TestPoint_Pad_D1.0mm, symbol Connector:TestPoint
- added TP11: VDD_3V3, pepy_sym_lib:[TEST_POINT]TestPoint_Pad_D1.0mm, symbol Connector:TestPoint
- added TP12: VBUS, pepy_sym_lib:[TEST_POINT]TestPoint_Pad_D1.0mm, symbol Connector:TestPoint
- added TP13: SIM_VCC, pepy_sym_lib:[TEST_POINT]TestPoint_Pad_D1.0mm, symbol Connector:TestPoint
- added TP14, TP8: VDD_COM, pepy_sym_lib:[TEST_POINT]TestPoint_Pad_D1.0mm, symbol Connector:TestPoint
- added TP9: VDD_AUX, pepy_sym_lib:[TEST_POINT]TestPoint_Pad_D1.0mm, symbol Connector:TestPoint
- R21, R22, R23, R24: now not fitted
Connections:
- net 1V8_COMM: now also TP10.1
- net DCOMM+: now also R29.2; no longer D3.4 (I/O2)
- net DCOMM-: now also R28.2; no longer D3.6 (I/O1)
- net GND: now also C28.1, D7.1 (C), D8.1 (C), D9.1 (C)
- net SIM_VCC: now also TP13.1
- net VBUS: now also C28.2, TP12.1
- net VDD_3V3: now also TP11.1
- net VDD_AUX: now also TP9.1
- net VDD_COMM: now also TP14.1, TP8.1
- net at C20.2, J8.1, L4.1: now also D9.2 (A)
- net at J5.1, R9.2: now also D7.2 (A)
- net at J6.1, R10.2: now also D8.2 (A)
- new net DR+: D3.4 (I/O2), R29.1
- new net DR-: D3.6 (I/O1), R28.1
Other:
- note added: "Antennas"
- note added: "Header"
- note removed: "VDD_3V3 hier ENable"
- title: (none) -> GNSS/LTE module
- moved on the sheet: C1, C10, C11, C12, C13, C14, C15, C16, C17, C18, C19, C2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

Commit message: Rev A
Parts:
- D3: Manufacturer (none) -> STMicroelectronics
- J7: Manufacturer (none) -> XUNPU
Changed lines of the file:
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@@
 			)
 		)
+		(property "Manufacturer" "XUNPU"
+			(at 251.46 150.368 0)
+			(effects
+				(font
+					(size 1.27 1.27)
+				)
+				(hide yes)
+			)
+		)
 		(pin "11"
 		)
@@
 			(effects
 				(font
+					(size 1.27 1.27)
+				)
+				(hide yes)
+			)
+		)
+		(property "Manufacturer" "STMicroelectronics"
+			(at 284.48 193.802 0)
+			(effects
+				(font
